File: led_drv_pmod.kicad_pcb (KiCad board)
At the start: 2 copper layers, 20.3 x 48.3 mm, 19 parts, among them J1 pmod, U1 LTC3206

Commit message: fixed block capacitor and i2c pull up
Parts:
- moved C4 33.7 mm to (83.9, 53.5)
- moved R2 11.5 mm to (90.0, 50.9), turned to 180 degrees
- turned R1 to 0 degrees
Routing:
- net GND: track 63.9 -> 24.5 mm, vias 7 -> 4
- net /scl: track 35.6 -> 9.15 mm
- net /sda: track 23.4 -> 19.8 mm
- net Net-(C4-Pad1): track 67.6 -> 65.1 mm
- net Net-(R3-Pad1): track 4.58 -> 5.81 mm
- net +3V3: track 40.6 -> 39.4 mm
- net Net-(R4-Pad1): track 9.62 -> 10.4 mm
