File: led_drv_pmod.kicad_sch (KiCad schematic)
At the start: 19 parts, among them J1 pmod, U1 LTC3206

Commit message: add screenshots
Other:
- company: (none) -> S59MZ
- title: (none) -> LTC3206 LED driver
